File: docs/Eagle/microBitNano/Backup/nanoController.brd (EAGLE design)
At the start: 67.4 x 79.9 mm, 35 parts, among them J17 IR RX, J18 IR RX, J19 IR RX, J2 MTXNRX, J20 IR RX, J21 IR RX, J22 IR RX, J23 IR RX, J24 IR RX, J3 IR RX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

Commit message: crossover
Parts:
- removed J26, J27: (no value), SparkFun-Connectors:1X01
- removed LED3: (no value), SparkFun-Connectors:1X04_LONGPADS
- removed R1, R2, R3: (no value), resistor-power:HPS58
Connections:
- removed net 3.3V: J10.1
- removed net D11: JP5.14
- removed net D12: JP5.15
- removed net N$1: LED3.4, R1.2
- removed net N$2: LED3.3, R2.2
- removed net N$3: LED3.1, R3.1
- net D2: no longer J26.1
- net D4: no longer R1.1
- net D7: no longer R2.1
- net D8: no longer R3.2
- net GND: no longer J27.1
- net M16: now also JP5.15
- net M8: now also JP5.14
- net VCC: now also J10.1, J5.P$1; no longer LED3.2
Routing:
- net D8: track 61.4 -> 0.00 mm
- net M16: track 157.9 -> 104.5 mm, vias 0 -> 1
- net VCC: track 128.8 -> 178.0 mm, vias 0 -> 1
- net D2: track 42.6 -> 0.00 mm
- net D7: track 35.1 -> 0.00 mm
- net D10: track 27.3 -> 51.0 mm
- net D4: track 21.4 -> 0.00 mm
- net D5: track 43.9 -> 62.3 mm, vias 1 -> 0
- net M6: track 37.7 -> 50.9 mm
- net N$2: track 12.7 -> 0.00 mm
- net D17: track 65.4 -> 55.7 mm, vias 1 -> 0
- net N$1: track 8.98 -> 0.00 mm
- net D6: track 58.1 -> 50.9 mm
- net M4: track 28.8 -> 35.9 mm, vias 1 -> 0
- net N$3: track 6.66 -> 0.00 mm
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Other:
- outline, holes or cut-outs redrawn
- board text removed: "D2"
