File: docs/Eagle/microBitNano/Backup/nanoController.sch (EAGLE design)
At the start: 35 parts, among them J17 IR RX, J18 IR RX, J19 IR RX, J2 MTXNRX, J20 IR RX, J21 IR RX, J22 IR RX, J23 IR RX, J24 IR RX, J3 IR RX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

Commit message: crossover
Parts:
- removed J26, J27: (no value), SparkFun-Connectors:CONN_01
- removed LED3: (no value), SparkFun-Connectors:CONN_04LONGPADS
- removed R1, R2, R3: (no value), resistor-power:RHPS58
Connections:
- removed net 3.3V: J10.1
- removed net D11: JP5.14
- removed net D12: JP5.15
- removed net N$1: LED3.4, R1.2
- removed net N$2: LED3.3, R2.2
- removed net N$3: LED3.1, R3.1
- net D2: no longer J26.1
- net D4: no longer R1.1
- net D7: no longer R2.1
- net D8: no longer R3.2
- net GND: no longer J27.1
- net M16: now also JP5.15
- net M8: now also JP5.14
- net VCC: now also J10.1, J5.1; no longer LED3.2
Other:
- note removed: "USB"
Changed lines of the file:
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@@
 <part name="P+14" library="SparkFun" deviceset="VCC" device=""/>
 <part name="J25" library="SparkFun-Connectors" deviceset="CONN_11" device=""/>
-<part name="LED3" library="SparkFun-Connectors" library_urn="urn:adsk.eagle:library:513" deviceset="CONN_04" device="LONGPADS" package3d_urn="urn:adsk.eagle:package:38098/1"/>
-<part name="P+15" library="SparkFun" deviceset="VCC" device=""/>
-<part name="J26" library="SparkFun-Connectors" deviceset="CONN_01" device=""/>
-<part name="J27" library="SparkFun-Connectors" deviceset="CONN_01" device=""/>
-<part name="GND21" library="SparkFun" deviceset="GND" device=""/>
-<part name="R1" library="resistor-power" library_urn="urn:adsk.eagle:library:344" deviceset="R" device="HPS58" package3d_urn="urn:adsk.eagle:package:25160/1"/>
-<part name="R2" library="resistor-power" library_urn="urn:adsk.eagle:library:344" deviceset="R" device="HPS58" package3d_urn="urn:adsk.eagle:package:25160/1"/>
-<part name="R3" library="resistor-power" library_urn="urn:adsk.eagle:library:344" deviceset="R" device="HPS58" package3d_urn="urn:adsk.eagle:package:25160/1"/>
 </parts>
 <sheets>
@@
 <text x="199.39" y="166.37" size="1.778" layer="91">Reset</text>
 <text x="203.2" y="138.43" size="1.778" layer="91">3V3</text>
-<text x="179.07" y="128.27" size="1.778" layer="91">USB</text>
 </plain>
 <instances>
@@
 <attribute name="NAME" x="40.64" y="163.068" size="1.778" layer="95" font="vector"/>
 </instance>
-<instance part="LED3" gate="G$1" x="181.61" y="223.52" smashed="yes" rot="R90">
-<attribute name="VALUE" x="188.976" y="218.44" size="1.778" layer="96" font="vector" rot="R90"/>
-<attribute name="NAME" x="173.482" y="218.44" size="1.778" layer="95" font="vector" rot="R90"/>
-</instance>
-<instance part="P+15" gate="1" x="181.61" y="236.22" smashed="yes">
-<attribute name="VALUE" x="180.594" y="239.776" size="1.778" layer="96"/>
-</instance>
-<instance part="J26" gate="G$1" x="-8.89" y="149.86" smashed="yes">
-<attribute name="VALUE" x="-11.43" y="145.034" size="1.778" layer="96" font="vector"/>
-<attribute name="NAME" x="-11.43" y="152.908" size="1.778" layer="95" font="vector"/>
-</instance>
-<instance part="J27" gate="G$1" x="-19.05" y="149.86" smashed="yes" rot="R180">
-<attribute name="VALUE" x="-16.51" y="154.686" size="1.778" layer="96" font="vector" rot="R180"/>
-<attribute name="NAME" x="-16.51" y="146.812" size="1.778" layer="95" font="vector" rot="R180"/>
-</instance>
-<instance part="GND21" gate="1" x="-33.02" y="147.32" smashed="yes">
-<attribute name="VALUE" x="-35.56" y="144.78" size="1.778" layer="96"/>
-</instance>
-<instance part="R1" gate="G$1" x="166.37" y="228.6" smashed="yes">
-<attribute name="NAME" x="162.56" y="229.9716" size="1.778" layer="95"/>
-<attribute name="VALUE" x="162.56" y="225.679" size="1.778" layer="96"/>
-</instance>
-<instance part="R2" gate="G$1" x="173.99" y="233.68" smashed="yes">
-<attribute name="NAME" x="170.18" y="235.0516" size="1.778" layer="95"/>
-<attribute name="VALUE" x="170.18" y="230.759" size="1.778" layer="96"/>
-</instance>
-<instance part="R3" gate="G$1" x="189.23" y="233.68" smashed="yes">
-<attribute name="NAME" x="185.42" y="235.0516" size="1.778" layer="95"/>
-<attribute name="VALUE" x="185.42" y="230.759" size="1.778" layer="96"/>
-</instance>
 </instances>
 <busses>
@@
 <wire x1="62.23" y1="384.81" x2="49.53" y2="384.81" width="0.1524" layer="91"/>
 </segment>
-<segment>
-<pinref part="J27" gate="G$1" pin="1"/>
-<pinref part="GND21" gate="1" pin="GND"/>
-<wire x1="-33.02" y1="149.86" x2="-26.67" y2="149.86" width="0.1524" layer="91"/>
-</segment>
 </net>
 <net name="D3" class="0">
@@
 <label x="158.75" y="148.59" size="1.778" layer="95"/>
 </segment>
-<segment>
-<pinref part="R2" gate="G$1" pin="1"/>
-<wire x1="168.91" y1="233.68" x2="157.48" y2="233.68" width="0.1524" layer="91"/>
-<label x="157.48" y="233.68" size="1.778" layer="95"/>
-</segment>
 </net>
 <net name="D8" class="0">
@@
 <label x="158.75" y="146.05" size="1.778" layer="95"/>
 </segment>
-<segment>
-<pinref part="R3" gate="G$1" pin="2"/>
-<wire x1="194.31" y1="233.68" x2="196.85" y2="233.68" width="0.1524" layer="91"/>
-<label x="196.85" y="233.68" size="1.778" layer="95"/>
-</segment>
 </net>
 <net name="D9" class="0">
@@
 </segment>
 <segment>
+<pinref part="J5" gate="G$1" pin="1"/>
+<pinref part="P+4" gate="1" pin="VCC"/>
+<wire x1="91.44" y1="208.28" x2="88.9" y2="208.28" width="0.1524" layer="91"/>
+</segment>
+<segment>
 <pinref part="J6" gate="G$1" pin="20"/>
 <pinref part="P+1" gate="1" pin="VCC"/>
@@
 </segment>
 <segment>
+<pinref part="J10" gate="G$1" pin="1"/>
+<pinref part="P+2" gate="1" pin="VCC"/>
+<wire x1="1.27" y1="171.45" x2="1.27" y2="181.61" width="0.1524" layer="91"/>
+</segment>
+<segment>
 <pinref part="J17" gate="J$1" pin="2"/>
 <pinref part="P+5" gate="1" pin="VCC"/>
@@
 <wire x1="57.15" y1="387.35" x2="49.53" y2="387.35" width="0.1524" layer="91"/>
 </segment>
-<segment>
-<pinref part="LED3" gate="G$1" pin="2"/>
-<pinref part="P+15" gate="1" pin="VCC"/>
-<wire x1="181.61" y1="236.22" x2="181.61" y2="228.6" width="0.1524" layer="91"/>
-</segment>
 </net>
 <net name="D4" class="0">
@@
 <label x="158.75" y="156.21" size="1.778" layer="95"/>
 </segment>
-<segment>
-<pinref part="R1" gate="G$1" pin="1"/>
-<wire x1="161.29" y1="228.6" x2="153.67" y2="228.6" width="0.1524" layer="91"/>
-<label x="153.67" y="228.6" size="1.778" layer="95"/>
-</segment>
 </net>
 <net name="D1" class="0">
@@
 <label x="158.75" y="161.29" size="1.778" layer="95"/>
 </segment>
-<segment>
-<pinref part="J26" gate="G$1" pin="1"/>
-<wire x1="-1.27" y1="149.86" x2="3.81" y2="149.86" width="0.1524" layer="91"/>
-<label x="3.81" y="149.86" size="1.778" layer="95"/>
-</segment>
 </net>
 <net name="D14" class="0">
@@
 <net name="M8" class="0">
 <segment>
+<pinref part="JP5" gate="G$1" pin="14"/>
+<wire x1="165.1" y1="138.43" x2="153.67" y2="138.43" width="0.1524" layer="91"/>
+<label x="153.67" y="138.43" size="1.778" layer="95"/>
+</segment>
+<segment>
 <pinref part="J6" gate="G$1" pin="11"/>
 <wire x1="50.8" y1="198.12" x2="59.69" y2="198.12" width="0.1524" layer="91"/>
@@
 <net name="M16" class="0">
 <segment>
+<pinref part="JP5" gate="G$1" pin="15"/>
+<wire x1="165.1" y1="135.89" x2="153.67" y2="135.89" width="0.1524" layer="91"/>
+<label x="153.67" y="135.89" size="1.778" layer="95"/>
+</segment>
+<segment>
 <pinref part="J6" gate="G$1" pin="3"/>
 <wire x1="50.8" y1="177.8" x2="59.69" y2="177.8" width="0.1524" layer="91"/>
@@
 </segment>
 </net>
-<net name="N$1" class="0">
-<segment>
-<pinref part="LED3" gate="G$1" pin="4"/>
-<pinref part="R1" gate="G$1" pin="2"/>
-<wire x1="171.45" y1="228.6" x2="176.53" y2="228.6" width="0.1524" layer="91"/>
-</segment>
-</net>
-<net name="N$2" class="0">
-<segment>
-<pinref part="LED3" gate="G$1" pin="3"/>
-<pinref part="R2" gate="G$1" pin="2"/>
-<wire x1="179.07" y1="233.68" x2="179.07" y2="228.6" width="0.1524" layer="91"/>
-</segment>
-</net>
-<net name="N$3" class="0">
-<segment>
-<pinref part="LED3" gate="G$1" pin="1"/>
-<pinref part="R3" gate="G$1" pin="1"/>
-<wire x1="184.15" y1="233.68" x2="184.15" y2="228.6" width="0.1524" layer="91"/>
-</segment>
-</net>
-<net name="D11" class="0">
-<segment>
-<pinref part="JP5" gate="G$1" pin="14"/>
-<wire x1="165.1" y1="138.43" x2="158.75" y2="138.43" width="0.1524" layer="91"/>
-<label x="158.75" y="138.43" size="1.778" layer="95"/>
-</segment>
-</net>
-<net name="D12" class="0">
-<segment>
-<pinref part="JP5" gate="G$1" pin="15"/>
-<wire x1="165.1" y1="135.89" x2="158.75" y2="135.89" width="0.1524" layer="91"/>
-<label x="158.75" y="135.89" size="1.778" layer="95"/>
-</segment>
-</net>
-<net name="3.3V" class="0">
-<segment>
-<pinref part="J10" gate="G$1" pin="1"/>
-<wire x1="1.27" y1="181.61" x2="7.62" y2="181.61" width="0.1524" layer="91"/>
-<label x="7.62" y="181.61" size="1.778" layer="95"/>
-</segment>
-</net>
