File: docs/Eagle/miniProIR/miniProIR.sch (EAGLE design)
At the start: 14 parts, among them J4 Pixel, J7 Interface

Commit message: Added spider/biped assembly
Parts:
- removed J3: (no value), SparkFun-Connectors:CONN_06SILK_FEMALE_PTH
Connections:
- net D0_E: no longer J3.4
- net D1_E: no longer J3.5
- net GND_E: no longer J3.2
- net VCC_E: no longer J3.3
Changed lines of the file:
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@@
 <part name="J1" library="SparkFun-Connectors" library_urn="urn:adsk.eagle:library:513" deviceset="CONN_12" device="" package3d_urn="urn:adsk.eagle:package:38169/1"/>
 <part name="J2" library="SparkFun-Connectors" library_urn="urn:adsk.eagle:library:513" deviceset="CONN_12" device="" package3d_urn="urn:adsk.eagle:package:38169/1"/>
-<part name="J3" library="SparkFun-Connectors" library_urn="urn:adsk.eagle:library:513" deviceset="CONN_06" device="SILK_FEMALE_PTH" package3d_urn="urn:adsk.eagle:package:38009/1"/>
 <part name="J4" library="SparkFun-Connectors" deviceset="CONN_03" device="" value="Pixel"/>
 <part name="J5" library="SparkFun-Connectors" deviceset="CONN_02" device=""/>
@@
 <attribute name="VALUE" x="323.596" y="372.11" size="1.778" layer="96" font="vector" rot="R90"/>
 <attribute name="NAME" x="287.782" y="372.11" size="1.778" layer="95" font="vector" rot="R90"/>
-</instance>
-<instance part="J3" gate="G$1" x="327.66" y="393.7" smashed="yes">
-<attribute name="VALUE" x="322.58" y="383.794" size="1.778" layer="96" font="vector"/>
-<attribute name="NAME" x="322.58" y="404.368" size="1.778" layer="95" font="vector"/>
 </instance>
 <instance part="J4" gate="J$1" x="293.37" y="431.8" smashed="yes" rot="R90">
@@
 </instance>
 <instance part="____1" gate="G$1" x="267.97" y="394.97" smashed="yes">
-<attribute name="NAME" x="270.51" y="384.9116" size="1.778" layer="95"/>
+<attribute name="NAME" x="264.16" y="388.7216" size="1.778" layer="95"/>
 <attribute name="VALUE" x="265.43" y="394.589" size="1.778" layer="96"/>
 </instance>
 <instance part="____2" gate="G$1" x="267.97" y="392.43" smashed="yes">
-<attribute name="NAME" x="270.51" y="382.3716" size="1.778" layer="95"/>
+<attribute name="NAME" x="264.16" y="386.1816" size="1.778" layer="95"/>
 <attribute name="VALUE" x="265.43" y="392.049" size="1.778" layer="96"/>
 </instance>
@@
 <wire x1="311.15" y1="408.94" x2="311.15" y2="400.05" width="0.1524" layer="91"/>
 <label x="311.15" y="400.05" size="1.778" layer="95" rot="R90"/>
-</segment>
-<segment>
-<pinref part="J3" gate="G$1" pin="2"/>
-<wire x1="332.74" y1="391.16" x2="334.01" y2="391.16" width="0.1524" layer="91"/>
-<label x="334.01" y="391.16" size="1.778" layer="95"/>
 </segment>
 <segment>
@@
 <wire x1="311.15" y1="382.27" x2="311.15" y2="384.81" width="0.1524" layer="91"/>
 <label x="311.15" y="384.81" size="1.778" layer="95" rot="R90"/>
-</segment>
-<segment>
-<pinref part="J3" gate="G$1" pin="3"/>
-<wire x1="332.74" y1="393.7" x2="334.01" y2="393.7" width="0.1524" layer="91"/>
-<label x="334.01" y="393.7" size="1.778" layer="95"/>
 </segment>
 <segment>
@@
 <net name="D0_E" class="0">
 <segment>
-<pinref part="J3" gate="G$1" pin="4"/>
-<wire x1="332.74" y1="396.24" x2="334.01" y2="396.24" width="0.1524" layer="91"/>
-<label x="334.01" y="396.24" size="1.778" layer="95"/>
-</segment>
-<segment>
 <pinref part="J1" gate="G$1" pin="11"/>
 <wire x1="316.23" y1="408.94" x2="316.23" y2="400.05" width="0.1524" layer="91"/>
@@
 <net name="D1_E" class="0">
 <segment>
-<pinref part="J3" gate="G$1" pin="5"/>
-<wire x1="332.74" y1="398.78" x2="334.01" y2="398.78" width="0.1524" layer="91"/>
-<label x="334.01" y="398.78" size="1.778" layer="95"/>
-</segment>
-<segment>
 <pinref part="J1" gate="G$1" pin="12"/>
