File: docs/Eagle/nxtMotorControl/nxtMini.sch (EAGLE design)
At the start: 18 parts, among them J11 RJ12, J3 RJ12, J7 Interface

Commit message: hyo
Parts:
- added J16, J17, J18, J19, J22, J24, J26, J28: 455-1750-1-ND, SparkFun-Connectors:CONN_03
- added J20, J21, J23, J25, J27, J29: (no value), SparkFun-Connectors:CONN_01
- J11, J3: value RJ12 -> 455-1750-1-ND; device con-rj:RJ12 -> SparkFun-Connectors:CONN_03
Connections:
- new net D4_E: 200.1, J1.6
- new net D7_E: J1.3, ____1.1
- new net D8_E: J1.2, ____2.1
- new net N$16: J19.1, J20.1
- new net N$17: J11.1, J21.1
- new net N$18: J22.1, J23.1
- new net N$19: J24.1, J25.1
- new net N$20: J26.1, J27.1
- new net N$21: J28.1, J29.1
- net D10_E: no longer ____2.1
- net D11_E: now also J7.1
- net D5_E: no longer 200.1
- net D6_E: no longer J7.1
- net D9_E: no longer ____1.1
- net N$1: now also J17.1; no longer J3.1
- net N$10: now also J14.2, J16.3; no longer J14.3, J3.5
- net N$11: now also J14.1, J17.3; no longer J14.4, J3.6
- net N$12: now also J15.4, J3.2; no longer J11.3, J15.1
- net N$13: now also J15.3, J18.2; no longer J11.4, J15.2
- net N$14: now also J15.2, J3.3; no longer J11.5, J15.3
- net N$15: now also J15.1, J18.3; no longer J11.6, J15.4
- net N$2: now also J16.1; no longer J3.2
- net N$6: now also J3.1; no longer J11.2
- net N$7: now also J18.1; no longer J11.1
- net N$8: now also J14.4, J16.2; no longer J14.1, J3.3
- net N$9: now also J14.3, J17.2; no longer J14.2, J3.4
Other:
- moved on the sheet: J10, J12, J13, J14, J15, J4
